Commit message: trying to fix local_costmap

File: src/cartographer_ros/cartographer_ros/urdf/00_Kobuki_rp.urdf (robot description, URDF)
Before this commit: robot ba_roboter, 5 links, 4 joints
Links:
- removed link base_footprint
- removed link rp_link
- added link base_link; visual box size=1 1 1
- added link laser; visual box size=0.1 0.1 0.1
Joints:
- joint base_joint: child base_footprint -> base_link; origin xyz=0 0 0.1 rpy=0 0 3.141 -> xyz=0 0 0.1 rpy=0 0 0; type fixed -> floating
- joint imu_joint: origin xyz=0 0 0 rpy=0 0 1.57 -> xyz=0 0 0 rpy=0 0 -1.57; parent base_footprint -> base_link
- joint rp_joint: child rp_link -> laser; origin xyz=0 0 0.2 rpy=0 0 0.0 -> xyz=0 0 0.2 rpy=0 0 -0.872655; parent base_footprint -> base_link

Commit message: updates from 2019_07_26

File: src/cartographer_ros/cartographer_ros/urdf/00_Kobuki_rp.urdf (robot description, URDF)
Before this commit: robot ba_roboter, 5 links, 4 joints
Links:
- removed link base_link
- removed link laser
- removed link map
- added link base_footprint; visual box size=1 1 1
- added link rp_link; visual box size=0.1 0.1 0.1
Joints:
- removed joint odom_joint
- joint base_joint: child base_link -> base_footprint; origin xyz=0 0 0.1 rpy=0 0 0 -> xyz=0 0 0.1 rpy=0 0 3.141
- joint imu_joint: parent base_link -> base_footprint
- joint rp_joint: child laser -> rp_link; parent base_link -> base_footprint

Commit message: optimized local planner

File: src/cartographer_ros/cartographer_ros/urdf/00_Kobuki_rp.urdf (robot description, URDF)
Before this commit: robot ba_roboter, 4 links, 3 joints
Joints:
- joint imu_joint: origin xyz=0 0 0 rpy=0 0 -1.57 -> xyz=0 0 0 rpy=0 0 +1.57
